File: pcb/MushyCloud.kicad_pcb (KiCad board)
At the start: 2 copper layers, 145.7 x 94.2 mm, 90 parts, among them J1 Conn_01x03_Male, J2 AudioJack3, J3 Conn_01x02_Male, J4 Conn_01x04_Male, J6 D2, SW1 SW_Push, SW10 SW_Push, SW11 SW_Push, SW12 SW_Push, SW13 SW_Push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

Commit message: final pcb release
Parts:
- added J4: Conn_01x04_Male, Connector_PinHeader_2.54mm:PinHeader_1x04_P2.54mm_Vertical, F.Cu at (184.9, 89.4)
- J2: value AudioJack3 -> Conn_01x04_Male; footprint MushyCloud:Jack_3.5mm_CUI_SJ-3523-SMT_Horizontal -> Connector_PinHeader_2.54mm:PinHeader_1x04_P2.54mm_Horizontal
- moved J2 6.89 mm to (180.5, 71.0), turned to 0 degrees
- moved J4 1.87 mm to (176.5, 89.5), turned to 65 degrees
Connections:
- U2 pad 1: Net-(U2-Pad1) -> tx
- U2 pad 2: data -> rx
Routing:
- net data: track 171.6 -> 0.00 mm, vias 3 -> 0
- net rx: track 0.00 -> 153.9 mm, vias 0 -> 2
- net tx: track 0.00 -> 150.4 mm, vias 0 -> 4
- net Net-(J4-Pad1): track 141.2 -> 153.8 mm
- net VCC: track 171.2 -> 168.3 mm
- net Net-(J4-Pad2): track 134.3 -> 137.0 mm
Other:
- board size 145.7 x 94.2 mm -> 143.5 x 94.2 mm
