File: pcb/MushyCloud.sch (KiCad schematic (older format))
At the start: 53 parts, among them J1 Conn_01x03_Male, J2 AudioJack3, J3 Conn_01x02_Male, J4 Conn_01x04_Male, SW1 SW_Push, SW10 SW_Push, SW11 SW_Push, SW12 SW_Push, SW13 SW_Push, SW14 SW_Push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

Commit message: final pcb release
Parts:
- removed J2: AudioJack3, MushyCloud:Jack_3.5mm_CUI_SJ-3523-SMT_Horizontal, symbol Connector:AudioJack3
- added J2: Conn_01x04_Male, Connector_PinHeader_2.54mm:PinHeader_1x04_P2.54mm_Horizontal, symbol Connector:Conn_01x04_Male
- U2: symbol keebio:ProMicro -> MushyCloud-components:ProMicro
Connections:
- net GND: now also J2.1 (Pin_1)
- net VCC: now also J2.2 (Pin_2)
- net tx: now reaches U2.1 (TX0/PD3)
- net tx: now also J2.3 (Pin_3)
- net data renamed rx
- net rx: now also J2.4 (Pin_4)
- no-connect marks 4 -> 3
Changed lines of the file:
@@
 $EndComp
 $Comp
-L keebio:ProMicro U2
+L MushyCloud-components:ProMicro U2
 U 1 1 5FECF752
 P 8900 2250
@@
 	1    0    0    -1
 $EndComp
-NoConn ~ 8200 1700
 NoConn ~ 9600 1700
 NoConn ~ 9600 2800
@@
 F 3 "" H 10200 850 50  0001 C CNN
 	1    10200 850
-	1    0    0    -1
-$EndComp
-Wire Wire Line
-	7700 4050 7400 4050
-Wire Wire Line
-	7400 4250 7700 4250
-$Comp
-L power:GND #PWR0108
-U 1 1 5FF3AE13
-P 7700 4250
-F 0 "#PWR0108" H 7700 4000 50  0001 C CNN
-F 1 "GND" H 7705 4077 50  0000 C CNN
-F 2 "" H 7700 4250 50  0001 C CNN
-F 3 "" H 7700 4250 50  0001 C CNN
-	1    7700 4250
-	1    0    0    -1
-$EndComp
-$Comp
-L power:VCC #PWR0109
-U 1 1 5FF3B352
-P 7700 4050
-F 0 "#PWR0109" H 7700 3900 50  0001 C CNN
-F 1 "VCC" H 7715 4223 50  0000 C CNN
-F 2 "" H 7700 4050 50  0001 C CNN
-F 3 "" H 7700 4050 50  0001 C CNN
-	1    7700 4050
 	1    0    0    -1
 $EndComp
@@
 Text GLabel 8200 2600 0    50   BiDi ~ 0
 row3
-Text GLabel 7550 1800 0    50   BiDi ~ 0
-data
-Wire Wire Line
-	7400 4150 7700 4150
-Text GLabel 7700 4150 2    50   BiDi ~ 0
-data
 $Comp
 L Switch:SW_Push SW22
@@
 Wire Wire Line
 	9600 1900 10050 1900
-Wire Wire Line
-	7550 1800 8200 1800
-$Comp
-L Connector:AudioJack3 J2
-U 1 1 5FFBBF42
-P 7200 4150
-F 0 "J2" H 7182 4475 50  0000 C CNN
-F 1 "AudioJack3" H 7182 4384 50  0000 C CNN
-F 2 "MushyCloud:Jack_3.5mm_CUI_SJ-3523-SMT_Horizontal" H 7200 4150 50  0001 C CNN
-F 3 "~" H 7200 4150 50  0001 C CNN
-	1    7200 4150
-	1    0    0    -1
-$EndComp
 $Comp
 L Connector:Conn_01x04_Male J4
@@
 Wire Wire Line
 	8200 2100 7050 2100
+Text GLabel 7550 1700 0    50   BiDi ~ 0
+tx
+Text GLabel 7550 1800 0    50   BiDi ~ 0
+rx
+Wire Wire Line
+	8200 1700 7550 1700
+Wire Wire Line
+	7550 1800 8200 1800
+Text GLabel 7100 3850 2    50   BiDi ~ 0
+tx
+Text GLabel 7100 3950 2    50   BiDi ~ 0
+rx
+$Comp
+L power:VCC #PWR0108
+U 1 1 5FFB0551
+P 7100 3750
+F 0 "#PWR0108" H 7100 3600 50  0001 C CNN
+F 1 "VCC" V 7115 3878 50  0000 L CNN
+F 2 "" H 7100 3750 50  0001 C CNN
+F 3 "" H 7100 3750 50  0001 C CNN
+	1    7100 3750
+	0    1    1    0
+$EndComp
+$Comp
+L power:GND #PWR0109
+U 1 1 5FFB105B
+P 7100 3650
+F 0 "#PWR0109" H 7100 3400 50  0001 C CNN
+F 1 "GND" V 7105 3522 50  0000 R CNN
+F 2 "" H 7100 3650 50  0001 C CNN
+F 3 "" H 7100 3650 50  0001 C CNN
+	1    7100 3650
+	0    -1   -1   0
+$EndComp
+$Comp
+L Connector:Conn_01x04_Male J2
+U 1 1 5FFFC688
+P 6900 3750
+F 0 "J2" H 7008 4031 50  0000 C CNN
+F 1 "Conn_01x04_Male" H 7008 3940 50  0000 C CNN
+F 2 "Connector_PinHeader_2.54mm:PinHeader_1x04_P2.54mm_Horizontal" H 6900 3750 50  0001 C CNN
+F 3 "~" H 6900 3750 50  0001 C CNN
+	1    6900 3750
+	1    0    0    -1
+$EndComp
 $EndSCHEMATC
